File: 001/001.sch (KiCad schematic (older format))
At the start: 17 parts, among them J1 To Pi, J2 POWER, J3 I2C 5V, J4 I2C 3.3V, SW1 SW_Push, SW2 SW_Push, SW3 SW_Push, U1 AE-PCA9306

Commit message: THD第1版
Parts:
- D1, D2, D3: footprint (none) -> LED_THT:LED_D3.0mm
- J1: footprint (none) -> Connector_JST:JST_XH_B12B-XH-A_1x12_P2.50mm_Vertical
- J2: footprint (none) -> Connector_JST:JST_XH_B2B-XH-A_1x02_P2.50mm_Vertical
- J3, J4: footprint (none) -> Connector_JST:JST_XH_B4B-XH-A_1x04_P2.50mm_Vertical
- R1, R2, R3, R4, R5, R6: footprint (none) -> Resistor_THT:R_Axial_DIN0309_L9.0mm_D3.2mm_P12.70mm_Horizontal
- SW1, SW2, SW3: footprint (none) -> HOLLY:TVDT18-050
- U1: footprint (none) -> Akizuki:AE-PCA9306; symbol 001-rescue:AE-PCA9306-Akizuki-001-rescue -> Akizuki:AE-PCA9306
Connections:
- wire segments 80 -> 79
- no-connect marks 1 -> 2
Other:
- moved on the sheet: J3, J4
