File: 001/001.kicad_pcb (KiCad board)
At the start: 2 copper layers, 59.7 x 40.6 mm, 33 parts, among them J1 To Pi, J2 POWER, J3 I2C 5V, J4 I2C 3.3V, SW1 SW_Push, SW2 SW_Push, SW3 SW_Push, U1 AE-PCA9306

Commit message: KiCAD 6
Routing:
- net GND: track 203.7 -> 0.00 mm
- net /GPIO05: track 0.00 -> 58.8 mm
- net /GPIO04: track 0.00 -> 39.6 mm
- net /+3.3V: track 0.00 -> 34.2 mm
- net Net-(D1-Pad2): track 39.2 -> 40.7 mm
- added copper zone on B.Cu, net GND
Other:
- net class Default removed

Commit message: 挿入実装初版完成
Routing:
- net /SDA: track 0.00 -> 104.0 mm, vias 0 -> 2
- net /SCL: track 0.00 -> 91.6 mm
- net /GPIO06: track 0.00 -> 76.7 mm
- net /+3.3V: track 34.2 -> 110.0 mm
- net Net-(J1-Pad9): track 0.00 -> 72.7 mm
- net /GPIO23: track 0.00 -> 64.9 mm
- net /GPIO24: track 0.00 -> 62.7 mm
- net Net-(D3-Pad2): track 0.00 -> 55.8 mm
- net /+5V: track 0.00 -> 45.4 mm
- net Net-(D2-Pad2): track 0.00 -> 24.0 mm
- net /SDA5V: track 0.00 -> 20.8 mm
- net /SCL5V: track 0.00 -> 14.3 mm
- net (no net): vias 0 -> 1
