File: 001/001.kicad_sch (KiCad schematic)
At the start: 17 parts

Commit message: 挿入実装初版完成
Parts:
- D1, D2: value (none) -> GREEN; footprint (none) -> LED_THT:LED_D3.0mm
- D3: value (none) -> RED; footprint (none) -> LED_THT:LED_D3.0mm
- J1: value (none) -> To Pi; footprint (none) -> Connector_JST:JST_XH_B12B-XH-A_1x12_P2.50mm_Vertical
- J2: value (none) -> POWER; footprint (none) -> Connector_JST:JST_XH_B2B-XH-A_1x02_P2.50mm_Vertical
- J3: value (none) -> I2C 5V; footprint (none) -> Connector_JST:JST_XH_B4B-XH-A_1x04_P2.50mm_Vertical
- J4: value (none) -> I2C 3.3V; footprint (none) -> Connector_JST:JST_XH_B4B-XH-A_1x04_P2.50mm_Vertical
- R1, R2, R3: value (none) -> 330; footprint (none) -> Resistor_THT:R_Axial_DIN0309_L9.0mm_D3.2mm_P12.70mm_Horizontal
- R4, R5, R6: value (none) -> 10k; footprint (none) -> Resistor_THT:R_Axial_DIN0309_L9.0mm_D3.2mm_P12.70mm_Horizontal
- SW1, SW2, SW3: value (none) -> SW_Push; footprint (none) -> HOLLY:TVDT18-050
- U1: value (none) -> AE-PCA9306; footprint (none) -> Akizuki:AE-PCA9306
